File: mk1/hardware/design/design.kicad_sch (KiCad schematic)
At the start: 34 parts, among them U1 Teensy4.1, U10 LIS2MDL, U11 TBC05-04, U12 TBC05-04, U2 HM-TRP-868, U3 BMP390, U4 LSM6DSV80X, U5 D30V30MAL, U6 L80-R, U7 VN5E160STR, U8 VN5E160STR, U9 TBC05-04

Commit message: First pass at PCB
Connections:
- net BMP-INT: now reaches U1.11 (9_OUT1C)
- net BMP-INT: now also U3.7 (INT)
- net BMP-CS: now reaches U1.12 (10_CS_MQSR)
- net BMP-CS: now also U3.6 (CSB)
- net MOSI: now reaches U1.13 (11_MOSI_CTX1)
- net MOSI: now also U3.4 (SDI), U4.14 (SDA)
- net MISO: now reaches U1.14 (12_MISO_MQSL)
- net MISO: now also U3.5 (SDO), U4.1 (SDO/TA0)
- net RF-TX: now reaches U1.16 (24_A10_TX6_SCL2)
- net RF-TX: now also U2.2 (DTX)
- net RF-RX: now reaches U1.17 (25_A11_RX6_SDA2)
- net RF-RX: now also U2.4 (DRX)
- net RF-CFG: now reaches U1.18 (26_A12_MOSI1)
- net RF-CFG: now also U2.5 (CONFIG)
- net RF-EN: now reaches U1.19 (27_A13_SCK1)
- net RF-EN: now also U2.6 (ENABLE)
- net APO-ON: now reaches U1.2 (0_RX1_CRX2_CS1)
- net APO-ON: now also U7.2 (INPUT)
- net GPS-TX: now reaches U1.20 (28_RX7)
- net GPS-TX: now also U6.2 (TXD1)
- net GPS-RX: now reaches U1.21 (29_TX7)
- net GPS-RX: now also U6.1 (RXD1)
- net GPS-1PPS: now reaches U1.22 (30_CRX3)
- net GPS-1PPS: now also U6.6 (1PPS)
- net GPS-RST: now reaches U1.23 (31_CTX3)
- net GPS-RST: now also U6.10 (~{RESET})
- net IMU-INT2: now reaches U1.26 (34_RX8)
- net IMU-INT2: now also U4.9 (INT2)
- net IMU-INT1: now reaches U1.27 (35_TX8)
- net IMU-INT1: now also U4.4 (INT1)
- net IMU-CS: now reaches U1.28 (36_CS)
- net IMU-CS: now also U4.12 (CS)
- net APO-STAT: now reaches U1.3 (1_TX1_CTX2_MISO1)
- net APO-STAT: now also R4.2, U7.3 (STATUS)
- net at U1.32 (40_A16): no longer BZ1.2 (-)
- net at U1.33 (41_A17): no longer BZ1.1 (+)
- net SCK: now reaches U1.35 (13_SCK_LED)
- net SCK: now also U3.2 (SCK), U4.13 (SCL)
- net MAIN-ON: now reaches U1.4 (2_OUT2)
- net MAIN-ON: now also U8.2 (INPUT)
- net SDA: now reaches U1.40 (18_A4_SDA)
- net SDA: now also R6.1, U10.4 (SDA/SDI/SDO)
- net SCL: now reaches U1.41 (19_A5_SCL)
- net SCL: now also R5.1, U10.1 (SCL/SPC)
- net MAG-DRDY: now reaches U1.43 (21_A7_RX5_BCLK1)
- net MAG-DRDY: now also U10.7 (DRDY)
- net at U1.44 (22_A8_CTX1): now also BZ1.2 (-)
- net at U1.45 (23_A9_CRX1_MCLK1): now also BZ1.1 (+)
- net MAIN-STAT: now reaches U1.5 (3_LRCLK2)
- net MAIN-STAT: now also R3.2, U8.3 (STATUS)
- net PWM1: now reaches U1.6 (4_BCLK2)
- net PWM1: now also U11.1 (1_VCC)
- net PWM2: now reaches U1.7 (5_IN2)
- net PWM2: now also U11.3 (2_VCC)
- net PWM3: now reaches U1.8 (6_OUT1D)
- net PWM3: now also U12.1 (1_VCC)
- net PWM4: now reaches U1.9 (7_RX2_OUT1A)
- net PWM4: now also U12.3 (2_VCC)
- net MAIN-OUT: now reaches U8.6 (OUTPUT)
- net MAIN-OUT: now also U8.7 (OUTPUT), U9.3 (2_VCC)
- net APO-OUT: now reaches U7.6 (OUTPUT)
- net APO-OUT: now also U7.7 (OUTPUT), U9.1 (1_VCC)
Other:
- moved on the sheet: BZ1, C13

Commit message: Fixed errors and some warnings
Parts:
- added H1, H2: MountingHole, MountingHole:MountingHole_2.7mm_M2.5, symbol Mechanical:MountingHole
Changed lines of the file:
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@@
+	)
+	(symbol
+		(lib_id "Mechanical:MountingHole")
+		(at 143.51 129.54 0)
+		(unit 1)
+		(exclude_from_sim no)
+		(in_bom no)
+		(on_board yes)
+		(dnp no)
+		(fields_autoplaced yes)
+		(property "Reference" "H2"
+			(at 146.05 128.2699 0)
+			(effects
+				(font
+					(size 1.27 1.27)
+				)
+				(justify left)
+			)
+		)
+		(property "Value" "MountingHole"
+			(at 146.05 130.8099 0)
+			(effects
+				(font
+					(size 1.27 1.27)
+				)
+				(justify left)
+			)
+		)
+		(property "Footprint" "MountingHole:MountingHole_2.7mm_M2.5"
+			(at 143.51 129.54 0)
+			(effects
+				(font
+					(size 1.27 1.27)
+				)
+				(hide yes)
+			)
+		)
+		(property "Datasheet" "~"
+			(at 143.51 129.54 0)
+			(effects
+				(font
+					(size 1.27 1.27)
+				)
+				(hide yes)
+			)
+		)
+		(property "Description" "Mounting Hole without connection"
+			(at 143.51 129.54 0)
+			(effects
+				(font
+					(size 1.27 1.27)
+				)
+				(hide yes)
+			)
+		)
+		(instances
+			(project ""
+				(path "/7394b7e9-7fb5-4560-b644-53fc5f15190b"
+					(reference "H2")
+					(unit 1)
+				)
+			)
+		)
 	)
 	(symbol
@@
 					(unit 1)
 				)
+			)
+		)
+	)
+	(symbol
+		(lib_id "Mechanical:MountingHole")
+		(at 116.84 134.62 0)
+		(unit 1)
+		(exclude_from_sim no)
+		(in_bom no)
+		(on_board yes)
+		(dnp no)
+		(fields_autoplaced yes)
+		(property "Reference" "H1"
+			(at 119.38 133.3499 0)
+			(effects
+				(font
+					(size 1.27 1.27)
+				)
+				(justify left)
+			)
+		)
+		(property "Value" "MountingHole"
+			(at 119.38 135.8899 0)
+			(effects
+				(font
+					(size 1.27 1.27)
+				)
+				(justify left)
+			)
+		)
+		(property "Footprint" "MountingHole:MountingHole_2.7mm_M2.5"
+			(at 116.84 134.62 0)
+			(effects
+				(font
+					(size 1.27 1.27)
+				)
+				(hide yes)
+			)
+		)
+		(property "Datasheet" "~"
+			(at 116.84 134.62 0)
+			(effects
+				(font
+					(size 1.27 1.27)
+				)
+				(hide yes)
+			)
+		)
+		(property "Description" "Mounting Hole without connection"
+			(at 116.84 134.62 0)
+			(effects
+				(font
+					(size 1.27 1.27)
+				)
+				(hide yes)
+			)
+		)
+		(instances
+			(project ""
+				(path "/7394b7e9-7fb5-4560-b644-53fc5f15190b"
+					(reference "H1")
+					(unit 1)
+				)
